File: controll_8motor_dac_already_compl.brd (EAGLE design)
At the start: 101.6 x 73.3 mm, 60 parts

Commit message: version1 できた． なかなか配線がやばいものだなぁ．
Parts:
- moved DC-JACK 81.3 mm to (95.2, 20.3)
- moved ARDUINO-5V/GND 25.9 mm to (87.6, 48.3)
- moved ARDUINO5V/GND 25.5 mm to (92.7, 48.3)
- moved CHIPSELECT 16.1 mm to (87.6, 30.5)
- moved MCP3208‐1 5.68 mm to (45.7, 20.3), turned to 0 degrees
- moved ARDUINO11~1 5.08 mm to (92.7, 39.4)
- moved ARDUINO11~13 5.08 mm to (87.6, 39.4)
- moved 安定化電源1 2.54 mm to (92.7, 59.7)
Routing:
- net P-DIORD1: track 0.00 -> 440.4 mm
- net ARDUINO-5V/GND: track 0.00 -> 237.4 mm
- net N$97: track 0.00 -> 191.2 mm
- net N$25: track 0.00 -> 120.5 mm
- net N$38: track 0.00 -> 115.0 mm
- net N$33: track 0.00 -> 100.7 mm
- net N$39: track 0.00 -> 68.9 mm
- net N$42: track 0.00 -> 63.0 mm
- net N$59: track 0.00 -> 44.4 mm
- net N$53: track 0.00 -> 40.7 mm
- net N$44: track 0.00 -> 37.2 mm
- net N$16: track 0.00 -> 36.4 mm
- net N$14: track 0.00 -> 36.0 mm
- net N$15: track 0.00 -> 35.9 mm
- net N$29: track 0.00 -> 35.9 mm
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