File: controll_8motor_dac_already_compl.sch (EAGLE design)
At the start: 60 parts

Commit message: version1 できた． なかなか配線がやばいものだなぁ．
Parts:
- DC-JACK: device BD6211F:JACK-PLUG0 -> con-jack:JACK-PLUG0
Connections:
- net N$26: now also LTC1660_1.13; no longer LTC1660_1.14
- net N$3: now also LTC1660_1.14; no longer LTC1660_1.13
Changed lines of the file:
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@@
 <part name="R16" library="rcl" library_urn="urn:adsk.eagle:library:334" deviceset="R-EU_" device="0204/2V" package3d_urn="urn:adsk.eagle:package:23495/1" value="240"/>
 <part name="ARDUINO5V/GND" library="pinhead" library_urn="urn:adsk.eagle:library:325" deviceset="PINHD-1X2" device="" package3d_urn="urn:adsk.eagle:package:22435/2"/>
+<part name="DC-JACK" library="con-jack" library_urn="urn:adsk.eagle:library:154" deviceset="JACK-PLUG" device="0" package3d_urn="urn:adsk.eagle:package:7492/1"/>
 <part name="ARDUINO11~1" library="pinhead" library_urn="urn:adsk.eagle:library:325" deviceset="PINHD-1X3" device="" package3d_urn="urn:adsk.eagle:package:22458/2"/>
 <part name="CHIPSELECT" library="pinhead" library_urn="urn:adsk.eagle:library:325" deviceset="PINHD-1X3" device="" package3d_urn="urn:adsk.eagle:package:22458/2"/>
@@
 <part name="M-DRIVER_6" library="BD6211F" deviceset="BD6211F-E2" device=""/>
 <part name="M-DRIVER_5" library="BD6211F" deviceset="BD6211F-E2" device=""/>
-<part name="DC-JACK" library="BD6211F" deviceset="JACK-PLUG" device="0" package3d_urn="urn:adsk.eagle:package:7492/1"/>
 </parts>
 <sheets>
@@
 <attribute name="VALUE" x="27.94" y="69.85" size="1.778" layer="96" rot="R90"/>
 </instance>
+<instance part="DC-JACK" gate="G$1" x="43.18" y="91.44" smashed="yes">
+<attribute name="NAME" x="33.02" y="96.52" size="1.778" layer="95"/>
+<attribute name="VALUE" x="35.56" y="86.36" size="1.778" layer="96"/>
+</instance>
 <instance part="ARDUINO11~1" gate="A" x="-50.8" y="116.84" smashed="yes" rot="R90">
 <attribute name="NAME" x="-56.515" y="110.49" size="1.778" layer="95" rot="R90"/>
@@
 <instance part="M-DRIVER_6" gate="G$1" x="-83.82" y="162.56" smashed="yes"/>
 <instance part="M-DRIVER_5" gate="G$1" x="-83.82" y="132.08" smashed="yes"/>
-<instance part="DC-JACK" gate="G$1" x="43.18" y="91.44" smashed="yes">
-<attribute name="NAME" x="35.56" y="96.52" size="1.778" layer="95"/>
-<attribute name="VALUE" x="35.56" y="86.36" size="1.778" layer="96"/>
-</instance>
 </instances>
 <busses>
@@
 <net name="N$3" class="0">
 <segment>
+<pinref part="LTC1660_1" gate="G$1" pin="14"/>
+<wire x1="-144.78" y1="200.66" x2="-137.16" y2="200.66" width="0.1524" layer="91"/>
+<wire x1="-144.78" y1="200.66" x2="-144.78" y2="220.98" width="0.1524" layer="91"/>
 <wire x1="-144.78" y1="220.98" x2="-200.66" y2="220.98" width="0.1524" layer="91"/>
 <pinref part="M-DRIVER_4" gate="G$1" pin="FIN"/>
 <wire x1="-200.66" y1="220.98" x2="-200.66" y2="228.6" width="0.1524" layer="91"/>
-<pinref part="LTC1660_1" gate="G$1" pin="13"/>
-<wire x1="-137.16" y1="203.2" x2="-144.78" y2="203.2" width="0.1524" layer="91"/>
-<wire x1="-144.78" y1="203.2" x2="-144.78" y2="220.98" width="0.1524" layer="91"/>
 </segment>
 </net>
@@
 <wire x1="22.86" y1="200.66" x2="43.18" y2="200.66" width="0.1524" layer="91"/>
 <junction x="43.18" y="200.66"/>
+<pinref part="DC-JACK" gate="G$1" pin="3"/>
 <wire x1="48.26" y1="93.98" x2="43.18" y2="93.98" width="0.1524" layer="91"/>
 <wire x1="43.18" y1="93.98" x2="43.18" y2="106.68" width="0.1524" layer="91"/>
 <junction x="43.18" y="106.68"/>
-<pinref part="DC-JACK" gate="G$1" pin="3"/>
 </segment>
 </net>
@@
 <pinref part="P-DIODE8" gate="G$1" pin="1"/>
 <wire x1="53.34" y1="200.66" x2="60.96" y2="200.66" width="0.1524" layer="91"/>
+<pinref part="DC-JACK" gate="G$1" pin="1"/>
+<wire x1="48.26" y1="88.9" x2="58.42" y2="88.9" width="0.1524" layer="91"/>
 <wire x1="58.42" y1="88.9" x2="58.42" y2="104.14" width="0.1524" layer="91"/>
 <pinref part="ARDUINO-5V/GND" gate="G$1" pin="2"/>
@@
 <wire x1="22.86" y1="91.44" x2="22.86" y2="88.9" width="0.1524" layer="91"/>
 <wire x1="22.86" y1="81.28" x2="22.86" y2="73.66" width="0.1524" layer="91"/>
-<wire x1="58.42" y1="88.9" x2="48.26" y2="88.9" width="0.1524" layer="91"/>
+<wire x1="48.26" y1="88.9" x2="22.86" y2="88.9" width="0.1524" layer="91"/>
+<junction x="48.26" y="88.9"/>
 <junction x="22.86" y="88.9"/>
 <pinref part="M-DRIVER_4" gate="G$1" pin="GND"/>
-<wire x1="48.26" y1="88.9" x2="22.86" y2="88.9" width="0.1524" layer="91"/>
 <wire x1="-167.64" y1="236.22" x2="-172.72" y2="236.22" width="0.1524" layer="91"/>
 <pinref part="M-DRIVER_3" gate="G$1" pin="GND"/>
@@
 <pinref part="M-DRIVER_5" gate="G$1" pin="GND"/>
 <wire x1="-66.04" y1="134.62" x2="-68.58" y2="134.62" width="0.1524" layer="91"/>
-<pinref part="DC-JACK" gate="G$1" pin="1"/>
-<junction x="48.26" y="88.9"/>
 </segment>
 </net>
@@
 <net name="N$26" class="0">
 <segment>
-<pinref part="LTC1660_1" gate="G$1" pin="14"/>
-<wire x1="-137.16" y1="200.66" x2="-170.18" y2="200.66" width="0.1524" layer="91"/>
-<wire x1="-170.18" y1="200.66" x2="-170.18" y2="198.12" width="0.1524" layer="91"/>
 <pinref part="M-DRIVER_3" gate="G$1" pin="RIN"/>
-<wire x1="-170.18" y1="198.12" x2="-172.72" y2="198.12" width="0.1524" layer="91"/>
-</segment>
-</net>
+<wire x1="-172.72" y1="198.12" x2="-170.18" y2="198.12" width="0.1524" layer="91"/>
+<wire x1="-170.18" y1="198.12" x2="-170.18" y2="203.2" width="0.1524" layer="91"/>
+<pinref part="LTC1660_1" gate="G$1" pin="13"/>
+<wire x1="-170.18" y1="203.2" x2="-137.16" y2="203.2" width="0.1524" layer="91"/>
+</segment>
+</net>
